File: BareDrones-FC-V1.kicad_pcb (KiCad board)
At the start: 6 copper layers, 37.1 x 37.2 mm, 128 parts, among them J10 Conn_01x08, J11 Conn_01x06, J12 Conn_01x06, J13 Conn_01x08, J14 Conn_01x02, J15 Conn_01x03, J16 Conn_01x03, J17 Conn_01x02, J18 USB4105-GF-A, J2 Conn_01x04, J20 Conn_02x07_Odd_Even, J3 Conn_01x04, J4 Conn_01x04, J5 Conn_01x04, J6 Conn_01x03, J7 Conn_01x04, J8 Conn_01x04, J9 Conn_01x04, Q1 BSS138, SW1 SW_Push, U1 STM32F722RETx, U2 MPU-6000, U3 BMP280, U4 W25Q128JVS, U5 MAX7456EUI+, U6 MP4560_QFN10, U7 LP2985-3.3, U8 LP2985-3.3, U9 MP4560_QFN10, Y1 CSTNE8M00G55Z000R0, Y2 27MHz

Commit message: Finished connections
Parts:
- removed L1: EGA, JPW_Footprints:EGA
- moved L2 20.9 mm to (103.1, 88.3)
- moved C14 4.02 mm to (106.6, 99.9), turned to -90 degrees
- moved C12 3.13 mm to (96.2, 87.3), turned to 180 degrees
- moved C2 1.67 mm to (88.0, 88.9), turned to 180 degrees
- moved C8 1.67 mm to (89.6, 88.3), turned to 90 degrees
- moved C3 0.25 mm to (101.4, 91.2)
- turned C5 to 180 degrees
Routing:
- net +3V3: track 27.0 -> 45.7 mm, vias 8 -> 22
- net /Gyro/REGOUT: track 3.82 -> 1.42 mm
- net GND: track 0.00 -> 0.76 mm, vias 0 -> 44
- net /Connectors/CURR: track 31.0 -> 31.5 mm
Other:
- board text added: "+9V GND TX2 VID"
- board text removed: "+9V GND TX1 VID"
